Commit message: Functional and ready to train lidar multi-agent environment

File: gym_drone/assets/assets/robot.urdf (robot description, URDF)
Before this commit: robot onshape, 5 links, 4 joints
Links:
- link ccwprop: mass 0.0045605471506329564937 -> 0.0045605471506329573611
- link ccwprop_2: mass 0.0045605471506329564937 -> 0.0045605471506329573611
- link cwprop: mass 0.0045608789483441887491 -> 0.0045608789483441878818
- link cwprop_2: mass 0.0045608789483441887491 -> 0.0045608789483441878818
Joints:
- joint ccw_back: origin xyz=0.050000000000000016653 0.050000000000000030531 -0.010000000000000000208 rpy=3.141592653589793116 -0 0 -> xyz=-0.050000000000000030531 0.050000000000000016653 -0.010000000000000000208 rpy=3.141592653589793116 -0 0
- joint ccw_front: origin xyz=-0.049999999999999981959 -0.050000000000000016653 -0.010000000000000000208 rpy=3.141592653589793116 -0 0 -> xyz=0.050000000000000023592 -0.049999999999999981959 -0.010000000000000000208 rpy=3.141592653589793116 -0 0
- joint cw_back: origin xyz=-0.05000000000000003747 0.049999999999999968081 -0.010000000000000000208 rpy=3.141592653589793116 -0 0 -> xyz=-0.049999999999999968081 -0.05000000000000003747 -0.010000000000000000208 rpy=3.141592653589793116 -0 0
- joint cw_front: origin xyz=0.050000000000000016653 -0.049999999999999988898 -0.010000000000000000208 rpy=3.141592653589793116 -0 0 -> xyz=0.049999999999999988898 0.050000000000000016653 -0.010000000000000000208 rpy=3.141592653589793116 -0 0
